File: vectron_handheld_pcb/vectron_handheld_pcb.sch (KiCad schematic (older format))
At the start: 18 parts

Commit message: Save progress.
Connections:
- net at U?.5 (PA3): now also J?.3 (Pin_3)
- net at U?.6 (PA4): now also J?.8 (Pin_8)
- net at U?.7 (PA5): now also J?.7 (Pin_7)
- net at U?.8 (PA6): now also J?.6 (Pin_6)
- net at U?.9 (PA7): now also J?.4 (Pin_4)
Other:
- moved on the sheet: U?
Changed lines of the file:
@@
 L 6502:W65C22SxP U?
 U 1 1 5F6BF957
-P 13250 11750
-F 0 "U?" H 13250 13381 50  0000 C CNN
-F 1 "W65C22SxP" H 13250 13290 50  0000 C CIB
-F 2 "" H 13250 11900 50  0001 C CNN
-F 3 "http://www.westerndesigncenter.com/wdc/documentation/w65c22.pdf" H 13250 11900 50  0001 C CNN
-	1    13250 11750
+P 13800 14750
+F 0 "U?" H 13800 16381 50  0000 C CNN
+F 1 "W65C22SxP" H 13800 16290 50  0000 C CIB
+F 2 "" H 13800 14900 50  0001 C CNN
+F 3 "http://www.westerndesigncenter.com/wdc/documentation/w65c22.pdf" H 13800 14900 50  0001 C CNN
+	1    13800 14750
 	1    0    0    -1
 $EndComp
@@
 	1    0    0    -1
 $EndComp
+Wire Wire Line
+	23450 17250 16650 17250
+Wire Wire Line
+	16650 17250 16650 14350
+Wire Wire Line
+	16650 14350 14400 14350
+Wire Wire Line
+	23450 17450 16350 17450
+Wire Wire Line
+	16350 17450 16350 14250
+Wire Wire Line
+	16350 14250 14400 14250
+Wire Wire Line
+	14400 14150 16100 14150
+Wire Wire Line
+	16100 14150 16100 17550
+Wire Wire Line
+	16100 17550 23450 17550
+Wire Wire Line
+	14400 14050 15950 14050
+Wire Wire Line
+	15950 14050 15950 17650
+Wire Wire Line
+	15950 17650 23450 17650
+Wire Wire Line
+	14400 13950 16900 13950
+Wire Wire Line
+	16900 13950 16900 17150
+Wire Wire Line
+	16900 17150 23450 17150
 $EndSCHEMATC

Commit message: Save progress.
Parts:
- added C? (x5): 102, symbol Device:C_Small
- added R? (x9): 10K, symbol Device:R
- added R? (x5): 3.3K, symbol Device:R
- SW?: value SW_Push_Dual -> UP
- SW?: value SW_Push_Dual -> DOWN
- SW?: value SW_Push_Dual -> LEFT
- SW?: value SW_Push_Dual -> RIGHT
- SW?: value SW_Push_Dual -> Fire
- SW?: value SW_Push_Dual -> RST
Connections:
- net labels added: +5V, GND
- wire segments 15 -> 179
Other:
- moved on the sheet: SW?, U?

Commit message: Schematic finished.
Parts:
- added BT?: Battery, symbol Device:Battery
- added C?: 220uF, symbol Device:CP
- added R? (x3): 3.3K, symbol Device:R
Connections:
- wire segments 179 -> 528
Other:
- moved on the sheet: SW?, U?

Commit message: Begin PCB layout.
Parts:
- BT1: renamed from BT?; footprint (none) -> Connector_PinHeader_2.54mm:PinHeader_1x02_P2.54mm_Vertical
- C1, C2, C3, C4, C5: renamed from C?; footprint (none) -> Capacitor_THT:C_Disc_D5.1mm_W3.2mm_P5.00mm
- C6: renamed from C?; footprint (none) -> Capacitor_THT:CP_Radial_D8.0mm_P5.00mm
- J1: renamed from J?; footprint (none) -> Connector_PinHeader_2.54mm:PinHeader_1x10_P2.54mm_Vertical
- R1, R10, R11, R12, R13, R14, R15, R16, R17, R2, R3, R4, R5, R6, R7, R8, R9: renamed from R?; footprint (none) -> Resistor_THT:R_Axial_DIN0207_L6.3mm_D2.5mm_P10.16mm_Horizontal
- SW1, SW2, SW3, SW4, SW5, SW6: renamed from SW?; footprint (none) -> Buttons_Switches_THT:SW_TH_Tactile_Omron_B3F-10xx
- U1, U4: renamed from U?; footprint (none) -> Socket:DIP_Socket-40_W11.9_W12.7_W15.24_W17.78_W18.5_3M_240-1280-00-0602J
- U10, U3, U8, U9: renamed from U?; footprint N14 -> Socket:DIP_Socket-14_W4.3_W5.08_W7.62_W10.16_W10.9_3M_214-3339-00-0602J
- U2, U6: renamed from U?; footprint (none) -> Socket:DIP_Socket-28_W11.9_W12.7_W15.24_W17.78_W18.5_3M_228-1277-00-0602J
- U5, U7: renamed from U?; footprint (none) -> Socket:DIP_Socket-20_W4.3_W5.08_W7.62_W10.16_W10.9_3M_220-3342-00-0602J
- Y1: renamed from Y?; footprint OSC_ECS-100AX-040 -> Oscillator:Oscillator_DIP-14
Connections:
- net +5V: now also BT1.1 (+), C6.1
- net GND: now also BT1.2 (-), C6.2
Other:
- moved on the sheet: BT1, C6
