File: vectron_handheld_pcb/vectron_handheld_pcb.kicad_pcb (KiCad board)
At the start: 4 copper layers, 344.2 x 233.7 mm, 42 parts, among them J1 Display, SW1 RST, SW2 LEFT, SW3 UP, SW4 DOWN, SW5 RIGHT, SW6 Fire, U1 W65C02SxP, U10 SN74HC08N, U2 AT28C256-15PU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

Commit message: Save PCB layout.
Parts:
- moved BT1 319.2 mm to (222.2, -5.08)
- moved C6 314.4 mm to (224.8, 15.2)
- moved U8 267.0 mm to (-11.4, 53.3), turned to 180 degrees
- moved U9 266.8 mm to (-19.1, 2.54)
- moved U10 260.3 mm to (47.0, 24.1)
- moved U4 222.6 mm to (165.1, 190.5), turned to 270 degrees
- moved R10 169.6 mm to (144.8, 213.4)
- moved R5 156.6 mm to (52.1, 189.2), turned to 180 degrees
- moved R3 137.2 mm to (184.2, 146.1), turned to 90 degrees
- moved R12 135.2 mm to (125.7, 176.5), turned to 180 degrees
- moved R15 133.2 mm to (97.8, 207.0), turned to 180 degrees
- moved Y1 114.3 mm to (139.7, 133.3)
- moved R13 113.8 mm to (97.8, 181.6), turned to 180 degrees
- moved SW6 101.9 mm to (199.4, 188.0)
- moved J1 99.1 mm to (26.7, 96.5)
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
Commit message: Finished routing.
Parts:
- moved R9 139.9 mm to (162.6, 73.7), turned to 270 degrees
- moved U4 117.1 mm to (139.7, 76.2), turned to 0 degrees
- moved U5 116.8 mm to (53.3, 5.08)
- moved R10 115.7 mm to (162.6, 99.1), turned to 90 degrees
- moved Y1 89.5 mm to (228.6, 123.2), turned to 180 degrees
- moved U7 75.1 mm to (73.7, 25.4)
- moved U10 74.7 mm to (-24.1, 47.0)
- moved R11 69.9 mm to (130.8, 111.8), turned to 270 degrees
- moved R12 58.4 mm to (125.7, 118.1), turned to 270 degrees
- moved U6 54.6 mm to (161.3, 21.6), turned to 0 degrees
- moved U8 49.8 mm to (-16.5, 102.9)
- moved U2 30.6 mm to (186.7, 21.6), turned to 0 degrees
- moved C2 17.8 mm to (57.1, 168.9)
- moved C3 17.8 mm to (82.5, 172.7)
- moved C4 17.8 mm to (57.1, 179.1)
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Routing:
- net Net-(U1-Pad25): track 0.00 -> 474.9 mm, vias 0 -> 4
- net Net-(U4-Pad23): track 0.00 -> 298.2 mm
- net Net-(U10-Pad2): track 0.00 -> 290.6 mm, vias 0 -> 2
- net Net-(U1-Pad16): track 0.00 -> 280.7 mm, vias 0 -> 4
- net GND: track 0.00 -> 275.7 mm, vias 0 -> 1
- net Net-(U1-Pad15): track 0.00 -> 274.8 mm, vias 0 -> 4
- net Net-(U1-Pad14): track 0.00 -> 271.3 mm, vias 0 -> 4
- net Net-(U6-Pad27): track 0.00 -> 267.0 mm, vias 0 -> 4
- net Net-(U1-Pad13): track 0.00 -> 266.6 mm, vias 0 -> 4
- net Net-(U2-Pad20): track 0.00 -> 256.2 mm, vias 0 -> 3
- net Net-(U1-Pad39): track 0.00 -> 256.1 mm
- net Net-(U1-Pad18): track 0.00 -> 254.8 mm, vias 0 -> 5
- net Net-(U1-Pad17): track 0.00 -> 251.2 mm, vias 0 -> 4
- net Net-(U1-Pad12): track 0.00 -> 246.5 mm, vias 0 -> 4
- net Net-(R12-Pad2): track 0.00 -> 245.7 mm
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
Commit message: Resize board..
Routing:
- net Net-(R10-Pad2): track 13.5 -> 231.9 mm, vias 0 -> 1
- net Net-(R6-Pad2): track 10.8 -> 195.9 mm
- net Net-(U1-Pad24): track 160.2 -> 244.7 mm, vias 1 -> 3
- net Net-(U1-Pad22): track 160.6 -> 217.6 mm, vias 1 -> 3
- net Net-(U1-Pad31): track 149.1 -> 198.7 mm, vias 0 -> 1
- net Net-(U1-Pad33): track 143.0 -> 192.3 mm
- net Net-(U1-Pad32): track 144.8 -> 193.4 mm
- net Net-(C3-Pad1): track 102.9 -> 106.5 mm
Other:
- board size 344.2 x 233.7 mm -> 273.1 x 221 mm
Changed lines of the file:
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@@
     (thickness 1.6)
     (drawings 4)
-    (tracks 817)
+    (tracks 875)
     (zones 0)
     (modules 42)
@@
     )
   )
-  (gr_line (start -31.75 -11.43) (end 312.42 -11.43) (layer Edge.Cuts) (width 0.1))
-  (gr_line (start 312.42 -11.43) (end 312.42 222.25) (layer Edge.Cuts) (width 0.1))
-  (gr_line (start -31.75 222.25) (end -31.75 -11.43) (layer Edge.Cuts) (width 0.1))
-  (gr_line (start 312.42 222.25) (end -31.75 222.25) (layer Edge.Cuts) (width 0.1))
+  (gr_line (start 237.49 -24.13) (end 237.49 196.85) (layer Edge.Cuts) (width 0.1))
+  (gr_line (start -35.56 -24.13) (end 237.49 -24.13) (layer Edge.Cuts) (width 0.1))
+  (gr_line (start -35.56 196.85) (end -35.56 -24.13) (layer Edge.Cuts) (width 0.1))
+  (gr_line (start 237.49 196.85) (end -35.56 196.85) (layer Edge.Cuts) (width 0.1))
   (segment (start 154.564879 18.373199) (end 154.564879 49.154879) (width 0.25) (layer F.Cu) (net 1))
   (segment (start 159.738195 13.199883) (end 154.564879 18.373199) (width 0.25) (layer F.Cu) (net 1))
@@
   (segment (start 0.394003 162.784999) (end 64.760001 162.784999) (width 0.25) (layer F.Cu) (net 5))
   (segment (start -5.08 164.52) (end -1.340998 164.52) (width 0.25) (layer F.Cu) (net 5))
+  (segment (start 82.55 172.72) (end 80.01 170.18) (width 0.25) (layer B.Cu) (net 5))
   (segment (start 58.5 172.72) (end 57.15 174.07) (width 0.25) (layer F.Cu) (net 6))
   (segment (start 67.31 172.72) (end 58.5 172.72) (width 0.25) (layer F.Cu) (net 6))
@@
   (segment (start 162.56 87.76863) (end 162.56 88.9) (width 0.25) (layer F.Cu) (net 18))
   (segment (start 154.94 78.74) (end 155.22 78.74) (width 0.25) (layer F.Cu) (net 18))
+  (via (at 147.32 78.74) (size 0.8) (drill 0.4) (layers F.Cu B.Cu) (net 18))
+  (segment (start 140.74501 85.31499) (end 147.32 78.74) (width 0.25) (layer B.Cu) (net 18))
+  (segment (start 138.987143 85.31499) (end 140.74501 85.31499) (width 0.25) (layer B.Cu) (net 18))
+  (segment (start 18.701999 113.574999) (end 110.727134 113.574999) (width 0.25) (layer B.Cu) (net 18))
+  (segment (start 41.91 171.45) (end 18.324999 147.864999) (width 0.25) (layer B.Cu) (net 18))
+  (segment (start 18.324999 113.951999) (end 18.701999 113.574999) (width 0.25) (layer B.Cu) (net 18))
+  (segment (start 18.324999 147.864999) (end 18.324999 113.951999) (width 0.25) (layer B.Cu) (net 18))
+  (segment (start 110.727134 113.574999) (end 138.987143 85.31499) (width 0.25) (layer B.Cu) (net 18))
+  (segment (start 147.32 78.74) (end 154.94 78.74) (width 0.25) (layer F.Cu) (net 18))
   (segment (start 53.34 170.18) (end 52.07 171.45) (width 0.25) (layer F.Cu) (net 19))
   (segment (start 67.31 170.18) (end 53.34 170.18) (width 0.25) (layer F.Cu) (net 19))
   (segment (start 154.94 76.2) (end 162.56 83.82) (width 0.25) (layer F.Cu) (net 20))
+  (segment (start 163.359999 84.619999) (end 162.56 83.82) (width 0.25) (layer B.Cu) (net 20))
+  (segment (start 163.685001 84.945001) (end 163.359999 84.619999) (width 0.25) (layer B.Cu) (net 20))
+  (segment (start 97.060001 185.275001) (end 163.685001 118.650001) (width 0.25) (layer B.Cu) (net 20))
+  (segment (start 163.685001 118.650001) (end 163.685001 84.945001) (width 0.25) (layer B.Cu) (net 20))
+  (segment (start 43.035001 185.275001) (end 97.060001 185.275001) (width 0.25) (layer B.Cu) (net 20))
+  (segment (start 41.91 184.15) (end 43.035001 185.275001) (width 0.25) (layer B.Cu) (net 20))
   (segment (start 53.20137 184.15) (end 52.07 184.15) (width 0.25) (layer F.Cu) (net 21))
   (segment (start 57.17 184.15) (end 53.20137 184.15) (width 0.25) (layer F.Cu) (net 21))
@@
   (segment (start 162.959999 -3.410001) (end 162.959999 23.710001) (width 0.25) (layer B.Cu) (net 41))
   (segment (start 162.56 -3.81) (end 162.959999 -3.410001) (width 0.25) (layer B.Cu) (net 41))
+  (via (at 181.61 58.42) (size 0.8) (drill 0.4) (layers F.Cu B.Cu) (net 41))
+  (segment (start 181.61 70.13) (end 181.61 58.42) (width 0.25) (layer F.Cu) (net 41))
+  (segment (start 186.41 74.93) (end 181.61 70.13) (width 0.25) (layer F.Cu) (net 41))
+  (segment (start 186.69 74.93) (end 186.41 74.93) (width 0.25) (layer F.Cu) (net 41))
+  (via (at 180.34 55.88) (size 0.8) (drill 0.4) (layers F.Cu B.Cu) (net 41))
+  (segment (start 181.61 57.15) (end 180.34 55.88) (width 0.25) (layer B.Cu) (net 41))
+  (segment (start 181.61 58.42) (end 181.61 57.15) (width 0.25) (layer B.Cu) (net 41))
+  (segment (start 185.44 24.13) (end 186.69 24.13) (width 0.25) (layer F.Cu) (net 41))
+  (segment (start 185.36499 24.20501) (end 185.44 24.13) (width 0.25) (layer F.Cu) (net 41))
+  (segment (start 185.36499 50.85501) (end 185.36499 24.20501) (width 0.25) (layer F.Cu) (net 41))
+  (segment (start 180.34 55.88) (end 185.36499 50.85501) (width 0.25) (layer F.Cu) (net 41))
   (via (at 210.82 39.37) (size 0.8) (drill 0.4) (layers F.Cu B.Cu) (net 42))
   (segment (start 201.93 39.37) (end 210.82 39.37) (width 0.25) (layer F.Cu) (net 42))
@@
   (segment (start 162.936999 -5.260001) (end 161.29 -3.613002) (width 0.25) (layer B.Cu) (net 45))
   (segment (start 163.83 -5.260001) (end 162.936999 -5.260001) (width 0.25) (layer B.Cu) (net 45))
+  (via (at 170.18 58.42) (size 0.8) (drill 0.4) (layers F.Cu B.Cu) (net 45))
+  (segment (start 170.18 60.177867) (end 170.18 58.42) (width 0.25) (layer F.Cu) (net 45))
+  (segment (start 188.01501 77.037143) (end 186.952877 75.97501) (width 0.25) (layer F.Cu) (net 45))
+  (segment (start 188.01501 79.93499) (end 188.01501 77.037143) (width 0.25) (layer F.Cu) (net 45))
+  (segment (start 185.977143 75.97501) (end 170.18 60.177867) (width 0.25) (layer F.Cu) (net 45))
+  (segment (start 186.952877 75.97501) (end 185.977143 75.97501) (width 0.25) (layer F.Cu) (net 45))
+  (segment (start 187.94 80.01) (end 188.01501 79.93499) (width 0.25) (layer F.Cu) (net 45))
+  (segment (start 186.69 80.01) (end 187.94 80.01) (width 0.25) (layer F.Cu) (net 45))
+  (via (at 172.72 20.32) (size 0.8) (drill 0.4) (layers F.Cu B.Cu) (net 45))
+  (segment (start 172.175001 20.864999) (end 172.72 20.32) (width 0.25) (layer B.Cu) (net 45))
+  (segment (start 172.175001 56.424999) (end 172.175001 20.864999) (width 0.25) (layer B.Cu) (net 45))
+  (segment (start 170.18 58.42) (end 172.175001 56.424999) (width 0.25) (layer B.Cu) (net 45))
+  (segment (start 185.42 20.32) (end 186.69 21.59) (width 0.25) (layer F.Cu) (net 45))
+  (segment (start 172.72 20.32) (end 185.42 20.32) (width 0.25) (layer F.Cu) (net 45))
   (via (at 208.28 29.21) (size 0.8) (drill 0.4) (layers F.Cu B.Cu) (net 46))
   (segment (start 201.93 29.21) (end 208.28 29.21) (width 0.25) (layer F.Cu) (net 46))
@@
   (segment (start 155.24 97.79) (end 185.44 97.79) (width 0.25) (layer F.Cu) (net 59))
   (segment (start 154.94 99.06) (end 154.94 98.09) (width 0.25) (layer F.Cu) (net 59))
+  (segment (start 188.01501 59.032503) (end 185.407507 56.425) (width 0.25) (layer B.Cu) (net 59))
+  (via (at 185.407507 56.425) (size 0.8) (drill 0.4) (layers F.Cu B.Cu) (net 59))
+  (segment (start 187.94 97.79) (end 188.01501 97.71499) (width 0.25) (layer B.Cu) (net 59))
+  (segment (start 188.01501 97.71499) (end 188.01501 59.032503) (width 0.25) (layer B.Cu) (net 59))
+  (segment (start 186.69 97.79) (end 187.94 97.79) (width 0.25) (layer B.Cu) (net 59))
+  (segment (start 185.44 52.07) (end 186.69 52.07) (width 0.25) (layer F.Cu) (net 59))
+  (segment (start 185.007508 56.025001) (end 185.007508 52.502492) (width 0.25) (layer F.Cu) (net 59))
+  (segment (start 185.007508 52.502492) (end 185.44 52.07) (width 0.25) (layer F.Cu) (net 59))
+  (segment (start 185.407507 56.425) (end 185.007508 56.025001) (width 0.25) (layer F.Cu) (net 59))
   (segment (start 156.814929 38.684929) (end 160.04 41.91) (width 0.25) (layer F.Cu) (net 60))
   (segment (start 156.814929 19.305199) (end 156.814929 38.684929) (width 0.25) (layer F.Cu) (net 60))
@@
   (segment (start 160.02 96.52) (end 160.02 100.33) (width 0.25) (layer B.Cu) (net 61))
   (segment (start 160.02 100.33) (end 186.69 100.33) (width 0.25) (layer F.Cu) (net 61))
+  (segment (start 159.620001 96.120001) (end 160.02 96.52) (width 0.25) (layer B.Cu) (net 61))
+  (segment (start 159.620001 49.949999) (end 159.620001 96.120001) (width 0.25) (layer B.Cu) (net 61))
+  (segment (start 160.04 49.53) (end 159.620001 49.949999) (width 0.25) (layer B.Cu) (net 61))
+  (segment (start 161.29 49.53) (end 160.04 49.53) (width 0.25) (layer B.Cu) (net 61))
   (segment (start 156.364919 40.774919) (end 160.04 44.45) (width 0.25) (layer F.Cu) (net 62))
   (segment (start 156.364919 19.118799) (end 156.364919 40.774919) (width 0.25) (layer F.Cu) (net 62))
@@
   (segment (start 157.48 93.98) (end 157.48 102.87) (width 0.25) (layer B.Cu) (net 63))
   (segment (start 157.48 102.87) (end 186.69 102.87) (width 0.25) (layer F.Cu) (net 63))
+  (segment (start 160.04 46.99) (end 157.48 49.55) (width 0.25) (layer B.Cu) (net 63))
+  (segment (start 157.48 49.55) (end 157.48 93.414315) (width 0.25) (layer B.Cu) (net 63))
+  (segment (start 161.29 46.99) (end 160.04 46.99) (width 0.25) (layer B.Cu) (net 63))
+  (segment (start 157.48 93.414315) (end 157.48 93.98) (width 0.25) (layer B.Cu) (net 63))
   (via (at 168.91 120.65) (size 0.8) (drill 0.4) (layers F.Cu B.Cu) (net 64))
   (segment (start 157.46 120.65) (end 168.91 120.65) (width 0.25) (layer F.Cu) (net 64))

Commit message: Add silk screen labels.
Other:
- board text added: "5V"
- board text added: "6502"
- board text added: "6522"
- board text added: "7404"
- board text added: "7408"
- board text added: "7414"
- board text added: "7432"
- board text added: "74682"
- board text added: "Crystal Oscillator"
- board text added: "Down"
- board text added: "Fire"
- board text added: "GND"
- board text added: "Left"
- board text added: "Nick Bild github.com/nickbild/vectron_handheld September 2020 v1.0"
- board text added: "RAM"
- board text added: "ROM"
- board text added: "Reset"
- board text added: "Right"
- board text added: "Up"
- board text added: "Vectron Handheld"
Changed lines of the file:
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@@
   (general
     (thickness 1.6)
-    (drawings 4)
+    (drawings 27)
     (tracks 875)
     (zones 0)
@@
       (outputformat 1)
       (mirror false)
-      (drillshape 1)
+      (drillshape 0)
       (scaleselection 1)
-      (outputdirectory ""))
+      (outputdirectory "gerber/"))
   )
   (net 0 "")
@@
     )
   )
+  (gr_text GND (at 222.25 1.27) (layer F.SilkS)
+    (effects (font (size 1 1) (thickness 0.15)))
+  )
+  (gr_text "Vectron\nHandheld" (at 152.4 175.26) (layer F.SilkS)
+    (effects (font (size 12.7 12.7) (thickness 0.531)))
+  )
+  (gr_text 5V (at 222.25 -8.89) (layer F.SilkS)
+    (effects (font (size 1 1) (thickness 0.15)))
+  )
+  (gr_text "Nick Bild\ngithub.com/nickbild/vectron_handheld\nSeptember 2020\nv1.0" (at 204.47 190.5) (layer F.SilkS)
+    (effects (font (size 1 1) (thickness 0.15)) (justify left))
+  )
+  (gr_text Reset (at 203.2 147.32) (layer F.SilkS)
+    (effects (font (size 1 1) (thickness 0.15)))
+  )
+  (gr_text Fire (at 201.93 166.37) (layer F.SilkS)
+    (effects (font (size 1 1) (thickness 0.15)))
+  )
+  (gr_text "Crystal Oscillator" (at 220.98 116.84) (layer F.SilkS)
+    (effects (font (size 1 1) (thickness 0.15)))
+  )
+  (gr_text 6502 (at 194.31 63.5) (layer F.SilkS)
+    (effects (font (size 1 1) (thickness 0.15)))
+  )
+  (gr_text ROM (at 194.31 7.62) (layer F.SilkS)
+    (effects (font (size 1 1) (thickness 0.15)))
+  )
+  (gr_text RAM (at 168.91 7.62) (layer F.SilkS)
+    (effects (font (size 1 1) (thickness 0.15)))
+  )
+  (gr_text 6522 (at 147.32 62.23) (layer F.SilkS)
+    (effects (font (size 1 1) (thickness 0.15)))
+  )
+  (gr_text 5V (at 21.59 86.36) (layer F.SilkS)
+    (effects (font (size 1 1) (thickness 0.15)))
+  )
+  (gr_text GND (at 21.59 83.82) (layer F.SilkS)
+    (effects (font (size 1 1) (thickness 0.15)))
+  )
+  (gr_text 74682 (at 63.5 19.05) (layer F.SilkS)
+    (effects (font (size 1 1) (thickness 0.15)))
+  )
+  (gr_text 74682 (at 63.5 -8.89) (layer F.SilkS)
+    (effects (font (size 1 1) (thickness 0.15)))
+  )
+  (gr_text 7432 (at -20.32 -10.16) (layer F.SilkS)
+    (effects (font (size 1 1) (thickness 0.15)))
+  )
+  (gr_text 7408 (at -20.32 33.02) (layer F.SilkS)
+    (effects (font (size 1 1) (thickness 0.15)))
+  )
+  (gr_text 7404 (at -20.32 77.47) (layer F.SilkS)
+    (effects (font (size 1 1) (thickness 0.15)))
+  )
+  (gr_text 7414 (at 71.12 153.67) (layer F.SilkS)
+    (effects (font (size 1 1) (thickness 0.15)))
+  )
+  (gr_text Right (at 8.89 166.37) (layer F.SilkS)
+    (effects (font (size 1 1) (thickness 0.15)))
+  )
+  (gr_text Left (at -12.7 166.37) (layer F.SilkS)
+    (effects (font (size 1 1) (thickness 0.15)))
+  )
+  (gr_text Down (at -2.54 176.53) (layer F.SilkS)
+    (effects (font (size 1 1) (thickness 0.15)))
+  )
+  (gr_text Up (at -1.27 156.21) (layer F.SilkS)
+    (effects (font (size 1 1) (thickness 0.15)))
+  )
   (gr_line (start 237.49 -24.13) (end 237.49 196.85) (layer Edge.Cuts) (width 0.1))
